Commit message: MRPT and ICP now work. Controllers broken

File: workspace/src/van_loading/description/urdf/idris.urdf.xacro (robot description, xacro)
@@ -115,8 +115,8 @@
       <type>transmission_interface/SimpleTransmission</type>
       <joint name="chassis_to_${prefix}_axle_joint">
+        <hardwareInterface>hardware_interface/PositionJointInterface</hardwareInterface>
 <!--
-        <hardwareInterface>hardware_interface/PositionJointInterface</hardwareInterface>
+        <hardwareInterface>hardware_interface/EffortJointInterface</hardwareInterface>
 -->
-        <hardwareInterface>hardware_interface/EffortJointInterface</hardwareInterface>
       </joint>
       <actuator name="${prefix}_steering_motor">
@@ -147,11 +147,12 @@
         </geometry>
       </collision>
+<!--
       <visual>
         <origin xyz="0 0 0" rpy="0 0 0"/>
-<!--        <geometry>
+        <geometry>
           <mesh filename="$(find van_loading)/description/meshes/hokuyo.dae"/>
         </geometry>
-        -->
       </visual>
+-->
       <inertial>
         <mass value="1e-5" />
